Commit message: Addition of base.xacro and wheels.xacro with entirely modular structure

File: home_custom_base_description/urdf/inc/base.xacro (robot description, xacro)
@@ -5,9 +5,20 @@
     <xacro:arg name="name" default="home_base"/>
     <xacro:macro name="home_base_description" params="prefix name">
+        <!-- Base dimensions -->
+        <xacro:property name="base_length" value="0.4"/>
+        <xacro:property name="base_width" value="0.4"/>
+        <xacro:property name="wheel_connector_z" value="-0.12"/>
+        <!-- Common wheel connector properties -->
+        <xacro:property name="wheel_connector_roll" value="-1.57"/>
+        <xacro:property name="wheel_connector_pitch" value="0.0"/>
+        <xacro:property name="wheel_connector_yaw" value="0.0"/>
+        <xacro:property name="wheel_connector_axis_x" value="0"/>
+        <xacro:property name="wheel_connector_axis_y" value="0"/>
+        <xacro:property name="wheel_connector_axis_z" value="1"/>
         <material name="gray">
             <color rgba="0.6 0.6 0.6 1"/>
         </material>
         <!-- Links -->
-        <link name="${prefix}base_link">
+        <link name="${prefix}_base_link">
             <visual>
                 <origin xyz="0 0 0" rpy="3.14 0 0"/>
@@ -24,29 +35,58 @@
             </collision>
         </link>
-        <link name="${prefix}base_footprint">
+        <link name="${prefix}_base_footprint">
             <visual>
-                <origin xyz="0.0 0.0 0.0" rpy="0.0 0.0 0.0"/>
+                <origin xyz="0 0 0" rpy="0 0 0"/>
                 <geometry>
-                    <box size="0.0 0.0 0.00"/>
+                    <box size="0 0 0"/>
                 </geometry>
                 <material name="gray"/>
             </visual>
             <collision>
-                <origin xyz="0.0 0 0.0" rpy="0.0 0.0 0.0"/>
+                <origin xyz="0 0 0" rpy="0 0 0"/>
                 <geometry>
-                    <box size="0.0 0.0 0.00"/>
+                    <box size="0 0 0"/>
                 </geometry>
             </collision>
             <inertial>
-                <origin xyz="0.0 0 0.0" rpy="0.0 0 0"/>
+                <origin xyz="0 0 0" rpy="0 0 0"/>
                 <mass value="10.5"/>
                 <inertia ixx="0.0001" ixy="0" ixz="0" iyy="0.0001" iyz="0" izz="0.0001"/>
             </inertial>
         </link>
-        <!-- Joints -->
-        <joint name="${prefix}base_link_joint" type="fixed">
-            <parent link="${prefix}base_footprint"/>
-            <child link="${prefix}base_link"/>
+        <!-- Wheel frames: no geometry for simplicity -->
+        <link name="${prefix}_rear_left_wheel_frame"/>
+        <link name="${prefix}_rear_right_wheel_frame"/>
+        <link name="${prefix}_front_left_wheel_frame"/>
+        <link name="${prefix}_front_right_wheel_frame"/>
+        <!-- Joints connecting wheels to base_link -->
+        <joint name="${prefix}_base_link_joint" type="fixed">
+            <parent link="${prefix}_base_footprint"/>
+            <child link="${prefix}_base_link"/>
             <origin xyz="0 0 0.2" rpy="0 0 0"/>
+        </joint>
+        <!-- Rear Left -->
+        <joint name="${prefix}_rear_left_wheel_joint" type="fixed">
+            <parent link="${prefix}_base_link"/>
+            <child link="${prefix}_rear_left_wheel_frame"/>
+            <origin xyz="${-(base_length / 2)} ${(base_width / 2)} ${wheel_connector_z}" rpy="${(wheel_connector_roll)} ${wheel_connector_pitch} ${wheel_connector_yaw}"/>
+        </joint>
+        <!-- Rear Right -->
+        <joint name="${prefix}_rear_right_wheel_joint" type="fixed">
+            <parent link="${prefix}_base_link"/>
+            <child link="${prefix}_rear_right_wheel_frame"/>
+            <origin xyz="${-(base_length / 2)} ${-(base_width / 2)} ${wheel_connector_z}" rpy="${-(wheel_connector_roll)} ${wheel_connector_pitch} ${wheel_connector_yaw}"/>
+        </joint>
+        <!-- Front Left -->
+        <joint name="${prefix}_front_left_wheel_joint" type="fixed">
+            <parent link="${prefix}_base_link"/>
+            <child link="${prefix}_front_left_wheel_frame"/>
+            <origin xyz="${(base_length / 2)} ${(base_width / 2)} ${wheel_connector_z}" rpy="${(wheel_connector_roll)} ${wheel_connector_pitch} ${wheel_connector_yaw}"/>
+        </joint>
+        <!-- Front Right -->
+        <joint name="${prefix}_front_right_wheel_joint" type="fixed">
+            <parent link="${prefix}_base_link"/>
+            <child link="${prefix}_front_right_wheel_frame"/>
+            <origin xyz="${(base_length / 2)} ${-(base_width / 2)} ${wheel_connector_z}" rpy="${-(wheel_connector_roll)} ${wheel_connector_pitch} ${wheel_connector_yaw}"/>
         </joint>
     </xacro:macro>

File: home_custom_base_description/urdf/robot.xacro (robot description, xacro)
@@ -1,9 +1,26 @@
 <?xml version="1.0"?>
-<robot name="home_base" xmlns:xacro="http://ros.org/wiki/xacro">
+<robot name="home_base"
+    xmlns:xacro="http://ros.org/wiki/xacro">
     <!-- Properties and Macros -->
-    <xacro:arg name="name" default="home_base"/>
-    <xacro:arg name="prefix" default=""/>
+    <xacro:property name="name" default="home_base"/>
+    <xacro:property name="prefix" default="home_base"/>
     <!-- Include base description -->
     <xacro:include filename="$(find home_custom_base_description)/urdf/inc/base.xacro"/>
-<xacro:home_base_description name="home_base" prefix="home_base_" />
+    <xacro:include filename="$(find home_custom_base_description)/urdf/inc/wheel.xacro"/>
+    <!-- Define base-->
+    <xacro:home_base_description name="${name}" prefix="${prefix}" />
+    <!-- Define wheel parent links -->
+    <xacro:property name="left_rear_parent_link" value="${prefix}_rear_left_wheel_frame"/>
+    <xacro:property name="right_rear_parent_link" value="${prefix}_rear_right_wheel_frame"/>
+    <xacro:property name="left_front_parent_link" value="${prefix}_front_left_wheel_frame"/>
+    <xacro:property name="right_front_parent_link" value="${prefix}_front_right_wheel_frame"/>
+    <!-- Define wheel connectors -->
+    <xacro:property name="connector_x_offset" value="0.0"/>
+    <xacro:property name="connector_y_offset" value="0.0"/>
+    <xacro:property name="connector_z_offset" value="0.015"/>
+    <!-- Define wheels -->
+    <xacro:home_base_wheel wheel_orientation="left" wheel_type="mecanum" parent_link="${left_rear_parent_link}" prefix="home_base_rear_left" x_offset="${connector_x_offset}" y_offset="${connector_y_offset}" z_offset="${connector_z_offset}" roll_offset="0.0" pitch_offset="0.0" yaw_offset="0.0" scale="0.001" axis_x="0" axis_y="0" axis_z="1" />
+    <xacro:home_base_wheel wheel_orientation="right" wheel_type="mecanum" parent_link="${right_rear_parent_link}" prefix="home_base_rear_right" x_offset="${connector_x_offset}" y_offset="${connector_y_offset}" z_offset="${connector_z_offset}" roll_offset="0.0" pitch_offset="0.0" yaw_offset="0.0" scale="0.001" axis_x="0" axis_y="0" axis_z="1" />
+    <xacro:home_base_wheel wheel_orientation="right" wheel_type="mecanum" parent_link="${right_front_parent_link}" prefix="home_base_front_right" x_offset="${connector_x_offset}" y_offset="${connector_y_offset}" z_offset="${connector_z_offset}" roll_offset="0.0" pitch_offset="0.0" yaw_offset="0.0" scale="0.001" axis_x="0" axis_y="0" axis_z="1" />
+    <xacro:home_base_wheel wheel_orientation="left" wheel_type="mecanum" parent_link="${left_front_parent_link}" prefix="home_base_front_left" x_offset="${connector_x_offset}" y_offset="${connector_y_offset}" z_offset="${connector_z_offset}" roll_offset="0.0" pitch_offset="0.0" yaw_offset="0.0" scale="0.001" axis_x="0" axis_y="0" axis_z="1" />
 </robot>

Commit message: Modifications to work with gazebo ign

File: home_custom_base_description/urdf/inc/base.xacro (robot description, xacro)
@@ -1,93 +1,90 @@
 <?xml version="1.0"?>
 <robot xmlns:xacro="http://ros.org/wiki/xacro">
-    <!-- Properties and Macros -->
-    <xacro:property name="mesh_dir" value="file://$(find home_custom_base_description)/meshes/collision"/>
-    <xacro:arg name="name" default="home_base"/>
-    <xacro:macro name="home_base_description" params="prefix name">
-        <!-- Base dimensions -->
-        <xacro:property name="base_length" value="0.4"/>
-        <xacro:property name="base_width" value="0.4"/>
-        <xacro:property name="wheel_connector_z" value="-0.12"/>
-        <!-- Common wheel connector properties -->
-        <xacro:property name="wheel_connector_roll" value="-1.57"/>
-        <xacro:property name="wheel_connector_pitch" value="0.0"/>
-        <xacro:property name="wheel_connector_yaw" value="0.0"/>
-        <xacro:property name="wheel_connector_axis_x" value="0"/>
-        <xacro:property name="wheel_connector_axis_y" value="0"/>
-        <xacro:property name="wheel_connector_axis_z" value="1"/>
-        <material name="gray">
-            <color rgba="0.6 0.6 0.6 1"/>
-        </material>
-        <!-- Links -->
-        <link name="${prefix}_base_link">
-            <visual>
-                <origin xyz="0 0 0" rpy="3.14 0 0"/>
-                <geometry>
-                    <mesh filename="${mesh_dir}/body.stl" scale="0.001 0.001 0.001"/>
-                </geometry>
-                <material name="gray"/>
-            </visual>
-            <collision>
-                <origin xyz="0 0 0" rpy="0 0 0"/>
-                <geometry>
-                    <mesh filename="${mesh_dir}/body.stl" scale="0.001 0.001 0.001"/>
-                </geometry>
-            </collision>
-        </link>
-        <link name="${prefix}_base_footprint">
-            <visual>
-                <origin xyz="0 0 0" rpy="0 0 0"/>
-                <geometry>
-                    <box size="0 0 0"/>
-                </geometry>
-                <material name="gray"/>
-            </visual>
-            <collision>
-                <origin xyz="0 0 0" rpy="0 0 0"/>
-                <geometry>
-                    <box size="0 0 0"/>
-                </geometry>
-            </collision>
-            <inertial>
-                <origin xyz="0 0 0" rpy="0 0 0"/>
-                <mass value="10.5"/>
-                <inertia ixx="0.0001" ixy="0" ixz="0" iyy="0.0001" iyz="0" izz="0.0001"/>
-            </inertial>
-        </link>
-        <!-- Wheel frames: no geometry for simplicity -->
-        <link name="${prefix}_rear_left_wheel_frame"/>
-        <link name="${prefix}_rear_right_wheel_frame"/>
-        <link name="${prefix}_front_left_wheel_frame"/>
-        <link name="${prefix}_front_right_wheel_frame"/>
-        <!-- Joints connecting wheels to base_link -->
-        <joint name="${prefix}_base_link_joint" type="fixed">
-            <parent link="${prefix}_base_footprint"/>
-            <child link="${prefix}_base_link"/>
-            <origin xyz="0 0 0.2" rpy="0 0 0"/>
-        </joint>
-        <!-- Rear Left -->
-        <joint name="${prefix}_rear_left_wheel_joint" type="fixed">
-            <parent link="${prefix}_base_link"/>
-            <child link="${prefix}_rear_left_wheel_frame"/>
-            <origin xyz="${-(base_length / 2)} ${(base_width / 2)} ${wheel_connector_z}" rpy="${(wheel_connector_roll)} ${wheel_connector_pitch} ${wheel_connector_yaw}"/>
-        </joint>
-        <!-- Rear Right -->
-        <joint name="${prefix}_rear_right_wheel_joint" type="fixed">
-            <parent link="${prefix}_base_link"/>
-            <child link="${prefix}_rear_right_wheel_frame"/>
-            <origin xyz="${-(base_length / 2)} ${-(base_width / 2)} ${wheel_connector_z}" rpy="${-(wheel_connector_roll)} ${wheel_connector_pitch} ${wheel_connector_yaw}"/>
-        </joint>
-        <!-- Front Left -->
-        <joint name="${prefix}_front_left_wheel_joint" type="fixed">
-            <parent link="${prefix}_base_link"/>
-            <child link="${prefix}_front_left_wheel_frame"/>
-            <origin xyz="${(base_length / 2)} ${(base_width / 2)} ${wheel_connector_z}" rpy="${(wheel_connector_roll)} ${wheel_connector_pitch} ${wheel_connector_yaw}"/>
-        </joint>
-        <!-- Front Right -->
-        <joint name="${prefix}_front_right_wheel_joint" type="fixed">
-            <parent link="${prefix}_base_link"/>
-            <child link="${prefix}_front_right_wheel_frame"/>
-            <origin xyz="${(base_length / 2)} ${-(base_width / 2)} ${wheel_connector_z}" rpy="${-(wheel_connector_roll)} ${wheel_connector_pitch} ${wheel_connector_yaw}"/>
-        </joint>
+  <!-- Properties and Macros -->
+  <xacro:property name="mesh_dir" value="file://$(find home_custom_base_description)/meshes/collision"/>
+  <xacro:arg name="name" default="home_base"/>
+  <xacro:macro name="home_base_description" params="prefix name">
+    <!-- Dimensions -->
+    <xacro:property name="base_length" value="0.4"/>
+    <xacro:property name="base_width" value="0.4"/>
+    <xacro:property name="wheel_connector_z" value="-0.12"/>
+    <xacro:property name="wheel_connector_roll" value="-1.57"/>
+    <xacro:property name="wheel_connector_pitch" value="0.0"/>
+    <xacro:property name="wheel_connector_yaw" value="0.0"/>
+    <xacro:property name="wheel_connector_axis_x" value="0"/>
+    <xacro:property name="wheel_connector_axis_y" value="0"/>
+    <xacro:property name="wheel_connector_axis_z" value="1"/>
+    <material name="gray">
+      <color rgba="0.6 0.6 0.6 1"/>
+    </material>
+    <!-- base_link -->
+    <link name="${prefix}_base_link">
+      <visual>
+        <origin xyz="0 0 0" rpy="3.14 0 0"/>
+        <geometry>
+          <mesh filename="${mesh_dir}/body.stl" scale="0.001 0.001 0.001"/>
+        </geometry>
+        <material name="gray"/>
+      </visual>
+      <collision>
+        <origin xyz="0 0 0" rpy="0 0 0"/>
+        <geometry>
+          <mesh filename="${mesh_dir}/body.stl" scale="0.001 0.001 0.001"/>
+        </geometry>
+      </collision>
+      <inertial>
+        <mass value="10.0"/>
+        <origin xyz="0 0 0" rpy="0 0 0"/>
+        <inertia ixx="0.01" ixy="0" ixz="0" iyy="0.01" iyz="0" izz="0.01"/>
+      </inertial>
+    </link>
+    <!-- base_footprint (no geometry, only inertial) -->
+    <link name="${prefix}_base_footprint">
+      <inertial>
+        <mass value="0.001"/>
+        <origin xyz="0 0 0" rpy="0 0 0"/>
+        <inertia ixx="0.00001" ixy="0" ixz="0" iyy="0.00001" iyz="0" izz="0.00001"/>
+      </inertial>
+    </link>
+    <!-- Empty frames for wheels -->
+    <xacro:macro name="empty_frame_link" params="link_name">
+      <link name="${link_name}">
+        <inertial>
+          <mass value="0.001"/>
+          <origin xyz="0 0 0" rpy="0 0 0"/>
+          <inertia ixx="0.00001" ixy="0" ixz="0" iyy="0.00001" iyz="0" izz="0.00001"/>
+        </inertial>
+      </link>
     </xacro:macro>
+    <xacro:empty_frame_link link_name="${prefix}_rear_left_wheel_frame"/>
+    <xacro:empty_frame_link link_name="${prefix}_rear_right_wheel_frame"/>
+    <xacro:empty_frame_link link_name="${prefix}_front_left_wheel_frame"/>
+    <xacro:empty_frame_link link_name="${prefix}_front_right_wheel_frame"/>
+    <!-- Fixed joints -->
+    <joint name="${prefix}_base_link_joint" type="fixed">
+      <parent link="${prefix}_base_footprint"/>
+      <child link="${prefix}_base_link"/>
+      <origin xyz="0 0 0.2" rpy="0 0 0"/>
+    </joint>
+    <joint name="${prefix}_rear_left_wheel_joint" type="fixed">
+      <parent link="${prefix}_base_link"/>
+      <child link="${prefix}_rear_left_wheel_frame"/>
+      <origin xyz="${-(base_length / 2)} ${(base_width / 2)} ${wheel_connector_z}" rpy="${wheel_connector_roll} ${wheel_connector_pitch} ${wheel_connector_yaw}"/>
+    </joint>
+    <joint name="${prefix}_rear_right_wheel_joint" type="fixed">
+      <parent link="${prefix}_base_link"/>
+      <child link="${prefix}_rear_right_wheel_frame"/>
+      <origin xyz="${-(base_length / 2)} ${-(base_width / 2)} ${wheel_connector_z}" rpy="${-wheel_connector_roll} ${wheel_connector_pitch} ${wheel_connector_yaw}"/>
+    </joint>
+    <joint name="${prefix}_front_left_wheel_joint" type="fixed">
+      <parent link="${prefix}_base_link"/>
+      <child link="${prefix}_front_left_wheel_frame"/>
+      <origin xyz="${(base_length / 2)} ${(base_width / 2)} ${wheel_connector_z}" rpy="${wheel_connector_roll} ${wheel_connector_pitch} ${wheel_connector_yaw}"/>
+    </joint>
+    <joint name="${prefix}_front_right_wheel_joint" type="fixed">
+      <parent link="${prefix}_base_link"/>
+      <child link="${prefix}_front_right_wheel_frame"/>
+      <origin xyz="${(base_length / 2)} ${-(base_width / 2)} ${wheel_connector_z}" rpy="${-wheel_connector_roll} ${wheel_connector_pitch} ${wheel_connector_yaw}"/>
+    </joint>
+  </xacro:macro>
 </robot>

File: home_custom_base_description/urdf/robot.xacro (robot description, xacro)
@@ -2,10 +2,20 @@
 <robot name="home_base"
     xmlns:xacro="http://ros.org/wiki/xacro">
+    <!-- Launch arguments -->
+    <xacro:arg name="use_sim_time" default="false"/>
+    <xacro:arg name="robot_type" default="real"/>
+    <xacro:arg name="prefix" default="home_base"/>
     <!-- Properties and Macros -->
     <xacro:property name="name" default="home_base"/>
-    <xacro:property name="prefix" default="home_base"/>
+    <xacro:property name="prefix" value="$(arg prefix)"/>
+    <xacro:property name="use_sim_time" value="$(arg use_sim_time)"/>
     <!-- Include base description -->
     <xacro:include filename="$(find home_custom_base_description)/urdf/inc/base.xacro"/>
     <xacro:include filename="$(find home_custom_base_description)/urdf/inc/wheel.xacro"/>
+    <!-- Conditionally include simulation files -->
+    <xacro:if value="${use_sim_time}">
+        <xacro:include filename="$(find home_custom_base_simulation)/urdf/home_base_ros2_control.xacro"/>
+        <xacro:include filename="$(find home_custom_base_simulation)/urdf/home_base_gazebo.xacro"/>
+    </xacro:if>
     <!-- Define base-->
     <xacro:home_base_description name="${name}" prefix="${prefix}" />
@@ -24,3 +34,10 @@
     <xacro:home_base_wheel wheel_orientation="right" wheel_type="mecanum" parent_link="${right_front_parent_link}" prefix="home_base_front_right" x_offset="${connector_x_offset}" y_offset="${connector_y_offset}" z_offset="${connector_z_offset}" roll_offset="0.0" pitch_offset="0.0" yaw_offset="0.0" scale="0.001" axis_x="0" axis_y="0" axis_z="1" />
     <xacro:home_base_wheel wheel_orientation="left" wheel_type="mecanum" parent_link="${left_front_parent_link}" prefix="home_base_front_left" x_offset="${connector_x_offset}" y_offset="${connector_y_offset}" z_offset="${connector_z_offset}" roll_offset="0.0" pitch_offset="0.0" yaw_offset="0.0" scale="0.001" axis_x="0" axis_y="0" axis_z="1" />
+    <!-- Conditionally add simulation components -->
+    <xacro:if value="${use_sim_time}">
+        <!-- Add ROS2 Control -->
+        <xacro:home_base_ros2_control name="${name}" prefix="${prefix}" use_sim_time="${use_sim_time}"/>
+        <!-- Add Gazebo simulation properties -->
+        <xacro:home_base_gazebo_sensors prefix="${prefix}"/>
+    </xacro:if>
 </robot>
