Commit message: fixed bad wheel kinematics

File: home_custom_base_description/urdf/home_base_ros2_control.xacro (robot description, xacro)
@@ -1,5 +1,6 @@
 <?xml version="1.0"?>
 <robot xmlns:xacro="http://ros.org/wiki/xacro">
-  <xacro:macro name="home_base_ros2_control" params="name prefix use_sim_time">
+  <xacro:macro name="home_base_ros2_control" params="name prefix use_sim_time"
+    xmlns:gz="http://gazebosim.org/schema">
     <!-- ROS 2 Control Setup - only for Gazebo simulation -->
     <xacro:if value="${use_sim_time}">
@@ -41,4 +42,59 @@
         </joint>
       </ros2_control>
+      <!-- To emulate Mecanum wheels in Gazebo with spherical collisions it
+  requires a custom friction model so the vehicle can strafe left to right -->
+      <!-- Wheel friction properties -->
+      <gazebo reference="${prefix}_rear_left_mecanum_left_wheel_link">
+        <collision>
+          <surface>
+            <friction>
+              <ode>
+                <mu>1.0</mu>
+                <mu2>0.0</mu2>
+                <fdir1 gz:expressed_in="base_link">1 -1 0</fdir1>
+              </ode>
+            </friction>
+          </surface>
+        </collision>
+      </gazebo>
+      <gazebo reference="${prefix}_rear_right_mecanum_right_wheel_link">
+        <collision>
+          <surface>
+            <friction>
+              <ode>
+                <mu>1.0</mu>
+                <mu2>0.0</mu2>
+                <fdir1 gz:expressed_in="base_link">1 -1 0</fdir1>
+              </ode>
+            </friction>
+          </surface>
+        </collision>
+      </gazebo>
+      <gazebo reference="${prefix}_front_left_mecanum_left_wheel_link">
+        <collision>
+          <surface>
+            <friction>
+              <ode>
+                <mu>1.0</mu>
+                <mu2>0.0</mu2>
+                <fdir1 gz:expressed_in="base_link">1 -1 0</fdir1>
+              </ode>
+            </friction>
+          </surface>
+        </collision>
+      </gazebo>
+      <gazebo reference="${prefix}_front_right_mecanum_right_wheel_link">
+        <collision>
+          <surface>
+            <friction>
+              <ode>
+                <mu>1.0</mu>
+                <mu2>0.0</mu2>
+                <fdir1 gz:expressed_in="base_link">1 -1 0</fdir1>
+              </ode>
+            </friction>
+          </surface>
+        </collision>
+      </gazebo>
       <!-- Gazebo ROS2 Control Plugin -->
       <gazebo>

File: home_custom_base_description/urdf/inc/base.xacro (robot description, xacro)
@@ -67,4 +67,5 @@
       <origin xyz="0 0 0.2" rpy="0 0 0"/>
     </joint>
+    <!-- Rear Left Wheel -->
     <joint name="${prefix}_rear_left_wheel_joint" type="fixed">
       <parent link="${prefix}_base_link"/>
@@ -72,9 +73,11 @@
       <origin xyz="${-(base_length / 2)} ${(base_width / 2)} ${wheel_connector_z}" rpy="${wheel_connector_roll} ${wheel_connector_pitch} ${wheel_connector_yaw}"/>
     </joint>
+    <!-- Rear Right Wheel (adjusted yaw angle for proper rotation) -->
     <joint name="${prefix}_rear_right_wheel_joint" type="fixed">
       <parent link="${prefix}_base_link"/>
       <child link="${prefix}_rear_right_wheel_frame"/>
-      <origin xyz="${-(base_length / 2)} ${-(base_width / 2)} ${wheel_connector_z}" rpy="${-wheel_connector_roll} ${wheel_connector_pitch} ${wheel_connector_yaw}"/>
+      <origin xyz="${-(base_length / 2)} ${-(base_width / 2)} ${wheel_connector_z}" rpy="${wheel_connector_roll} ${wheel_connector_pitch} ${wheel_connector_yaw}"/>
     </joint>
+    <!-- Front Left Wheel -->
     <joint name="${prefix}_front_left_wheel_joint" type="fixed">
       <parent link="${prefix}_base_link"/>
@@ -82,8 +85,9 @@
       <origin xyz="${(base_length / 2)} ${(base_width / 2)} ${wheel_connector_z}" rpy="${wheel_connector_roll} ${wheel_connector_pitch} ${wheel_connector_yaw}"/>
     </joint>
+    <!-- Front Right Wheel (adjusted yaw angle for proper rotation) -->
     <joint name="${prefix}_front_right_wheel_joint" type="fixed">
       <parent link="${prefix}_base_link"/>
       <child link="${prefix}_front_right_wheel_frame"/>
-      <origin xyz="${(base_length / 2)} ${-(base_width / 2)} ${wheel_connector_z}" rpy="${-wheel_connector_roll} ${wheel_connector_pitch} ${wheel_connector_yaw}"/>
+      <origin xyz="${(base_length / 2)} ${-(base_width / 2)} ${wheel_connector_z}" rpy="${wheel_connector_roll} ${wheel_connector_pitch} ${wheel_connector_yaw}"/>
     </joint>
   </xacro:macro>

File: home_custom_base_description/urdf/robot.xacro (robot description, xacro)
@@ -31,6 +31,6 @@
     <!-- Define wheels -->
     <xacro:home_base_wheel wheel_orientation="left" wheel_type="mecanum" parent_link="${left_rear_parent_link}" prefix="home_base_rear_left" x_offset="${connector_x_offset}" y_offset="${connector_y_offset}" z_offset="${connector_z_offset}" roll_offset="0.0" pitch_offset="0.0" yaw_offset="0.0" scale="0.001" axis_x="0" axis_y="0" axis_z="1" />
-    <xacro:home_base_wheel wheel_orientation="right" wheel_type="mecanum" parent_link="${right_rear_parent_link}" prefix="home_base_rear_right" x_offset="${connector_x_offset}" y_offset="${connector_y_offset}" z_offset="${connector_z_offset}" roll_offset="0.0" pitch_offset="0.0" yaw_offset="0.0" scale="0.001" axis_x="0" axis_y="0" axis_z="1" />
-    <xacro:home_base_wheel wheel_orientation="right" wheel_type="mecanum" parent_link="${right_front_parent_link}" prefix="home_base_front_right" x_offset="${connector_x_offset}" y_offset="${connector_y_offset}" z_offset="${connector_z_offset}" roll_offset="0.0" pitch_offset="0.0" yaw_offset="0.0" scale="0.001" axis_x="0" axis_y="0" axis_z="1" />
+    <xacro:home_base_wheel wheel_orientation="right" wheel_type="mecanum" parent_link="${right_rear_parent_link}" prefix="home_base_rear_right" x_offset="${connector_x_offset}" y_offset="${connector_y_offset}" z_offset="${-connector_z_offset}" roll_offset="0.0" pitch_offset="0.0" yaw_offset="0.0" scale="0.001" axis_x="0" axis_y="0" axis_z="1" />
+    <xacro:home_base_wheel wheel_orientation="right" wheel_type="mecanum" parent_link="${right_front_parent_link}" prefix="home_base_front_right" x_offset="${connector_x_offset}" y_offset="${connector_y_offset}" z_offset="${-connector_z_offset}" roll_offset="0.0" pitch_offset="0.0" yaw_offset="0.0" scale="0.001" axis_x="0" axis_y="0" axis_z="1" />
     <xacro:home_base_wheel wheel_orientation="left" wheel_type="mecanum" parent_link="${left_front_parent_link}" prefix="home_base_front_left" x_offset="${connector_x_offset}" y_offset="${connector_y_offset}" z_offset="${connector_z_offset}" roll_offset="0.0" pitch_offset="0.0" yaw_offset="0.0" scale="0.001" axis_x="0" axis_y="0" axis_z="1" />
     <!-- Conditionally add simulation components -->

Commit message: Fixed controller not loading

File: home_custom_base_description/urdf/home_base_ros2_control.xacro (robot description, xacro)
@@ -17,5 +17,5 @@
           <state_interface name="position"/>
         </joint>
-        <joint name="${prefix}_rear_left_mecanum_left_wheel_joint">
+        <joint name="${prefix}_rear_left_mecanum_right_wheel_joint">
           <command_interface name="velocity">
             <param name="min">-10</param>
@@ -33,5 +33,5 @@
           <state_interface name="position"/>
         </joint>
-        <joint name="${prefix}_rear_right_mecanum_right_wheel_joint">
+        <joint name="${prefix}_rear_right_mecanum_left_wheel_joint">
           <command_interface name="velocity">
             <param name="min">-10</param>

Commit message: Fixed wheel visual orientation issue

File: home_custom_base_description/urdf/home_base_ros2_control.xacro (robot description, xacro)
@@ -9,5 +9,5 @@
           <plugin>gz_ros2_control/GazeboSimSystem</plugin>
         </hardware>
-        <joint name="${prefix}_front_left_mecanum_left_wheel_joint">
+        <joint name="${prefix}_front_left_mecanum_right_wheel_joint">
           <command_interface name="velocity">
             <param name="min">-10</param>
@@ -17,5 +17,5 @@
           <state_interface name="position"/>
         </joint>
-        <joint name="${prefix}_rear_left_mecanum_right_wheel_joint">
+        <joint name="${prefix}_rear_left_mecanum_left_wheel_joint">
           <command_interface name="velocity">
             <param name="min">-10</param>
@@ -25,5 +25,5 @@
           <state_interface name="position"/>
         </joint>
-        <joint name="${prefix}_front_right_mecanum_right_wheel_joint">
+        <joint name="${prefix}_front_right_mecanum_left_wheel_joint">
           <command_interface name="velocity">
             <param name="min">-10</param>
@@ -33,5 +33,5 @@
           <state_interface name="position"/>
         </joint>
-        <joint name="${prefix}_rear_right_mecanum_left_wheel_joint">
+        <joint name="${prefix}_rear_right_mecanum_right_wheel_joint">
           <command_interface name="velocity">
             <param name="min">-10</param>

File: home_custom_base_description/urdf/robot.xacro (robot description, xacro)
@@ -30,8 +30,8 @@
     <xacro:property name="connector_z_offset" value="0.015"/>
     <!-- Define wheels -->
-    <xacro:home_base_wheel wheel_orientation="right" wheel_type="mecanum" parent_link="${left_rear_parent_link}" prefix="home_base_rear_left" x_offset="${connector_x_offset}" y_offset="${connector_y_offset}" z_offset="${connector_z_offset}" roll_offset="0.0" pitch_offset="0.0" yaw_offset="0.0" scale="0.001" axis_x="0" axis_y="0" axis_z="1" />
-    <xacro:home_base_wheel wheel_orientation="left" wheel_type="mecanum" parent_link="${right_rear_parent_link}" prefix="home_base_rear_right" x_offset="${connector_x_offset}" y_offset="${connector_y_offset}" z_offset="${-connector_z_offset}" roll_offset="0.0" pitch_offset="0.0" yaw_offset="0.0" scale="0.001" axis_x="0" axis_y="0" axis_z="1" />
-    <xacro:home_base_wheel wheel_orientation="right" wheel_type="mecanum" parent_link="${right_front_parent_link}" prefix="home_base_front_right" x_offset="${connector_x_offset}" y_offset="${connector_y_offset}" z_offset="${-connector_z_offset}" roll_offset="0.0" pitch_offset="0.0" yaw_offset="0.0" scale="0.001" axis_x="0" axis_y="0" axis_z="1" />
-    <xacro:home_base_wheel wheel_orientation="left" wheel_type="mecanum" parent_link="${left_front_parent_link}" prefix="home_base_front_left" x_offset="${connector_x_offset}" y_offset="${connector_y_offset}" z_offset="${connector_z_offset}" roll_offset="0.0" pitch_offset="0.0" yaw_offset="0.0" scale="0.001" axis_x="0" axis_y="0" axis_z="1" />
+    <xacro:home_base_wheel wheel_orientation="left" wheel_type="mecanum" parent_link="${left_rear_parent_link}" prefix="home_base_rear_left" x_offset="${connector_x_offset}" y_offset="${connector_y_offset}" z_offset="${connector_z_offset}" roll_offset="0.0" pitch_offset="0.0" yaw_offset="0.0" scale="0.001" axis_x="0" axis_y="0" axis_z="1" />
+    <xacro:home_base_wheel wheel_orientation="right" wheel_type="mecanum" parent_link="${right_rear_parent_link}" prefix="home_base_rear_right" x_offset="${connector_x_offset}" y_offset="${connector_y_offset}" z_offset="${-connector_z_offset}" roll_offset="0.0" pitch_offset="0.0" yaw_offset="0.0" scale="0.001" axis_x="0" axis_y="0" axis_z="1" />
+    <xacro:home_base_wheel wheel_orientation="left" wheel_type="mecanum" parent_link="${right_front_parent_link}" prefix="home_base_front_right" x_offset="${connector_x_offset}" y_offset="${connector_y_offset}" z_offset="${-connector_z_offset}" roll_offset="0.0" pitch_offset="0.0" yaw_offset="0.0" scale="0.001" axis_x="0" axis_y="0" axis_z="1" />
+    <xacro:home_base_wheel wheel_orientation="right" wheel_type="mecanum" parent_link="${left_front_parent_link}" prefix="home_base_front_left" x_offset="${connector_x_offset}" y_offset="${connector_y_offset}" z_offset="${connector_z_offset}" roll_offset="0.0" pitch_offset="0.0" yaw_offset="0.0" scale="0.001" axis_x="0" axis_y="0" axis_z="1" />
     <!-- Conditionally add simulation components -->
     <xacro:if value="${use_sim_time}">
