Commit message: Replace base URDF with SolidWorks-exported ensamblaje_v2 model
- Convert SolidWorks ROS1 export into parametric robot.xacro with
  prefix/use_sim_time/robot_type args
- Add base_footprint root (Z=0.0385 below base_link, matches 3" wheel radius)
- Fix wheel_RL axis (was 0 1 0, now 0 0 1 like the other wheels)
- Drop xarm link (mesh from exporter was an 80-byte placeholder)
- Move new visual meshes to meshes/visual/, drop unused collision meshes
- Update ros2_control joints to wheel_FL/FR/RL/RR
- Update Gazebo friction references to new wheel link names
  (home_base_wheel_FL/FR/RL/RR)
- Fix launch arg typo (decription_file -> description_file) and rename
  tf_prefix to prefix to match xacro; add use_gui toggle
- Reset rviz config (Fixed Frame: home_base_base_footprint)
- Remove dead code: urdf/inc/, xacro/ duplicate, home_base_gazebo.xacro

Cherry-picked from webots_sim 8a5a789 with extra friction reference fixes
to keep gz_ros2_control working on the new wheel naming.

Co-Authored-By: Claude Opus 4.7 <noreply@anthropic.com>

File: home_custom_base_description/urdf/home_base_ros2_control.xacro (robot description, xacro)
@@ -9,5 +9,5 @@
           <plugin>gz_ros2_control/GazeboSimSystem</plugin>
         </hardware>
-        <joint name="${prefix}_front_left_mecanum_right_wheel_joint">
+        <joint name="${prefix}_wheel_FL_joint">
           <command_interface name="velocity">
             <param name="min">-10</param>
@@ -17,5 +17,5 @@
           <state_interface name="position"/>
         </joint>
-        <joint name="${prefix}_rear_left_mecanum_left_wheel_joint">
+        <joint name="${prefix}_wheel_FR_joint">
           <command_interface name="velocity">
             <param name="min">-10</param>
@@ -25,5 +25,5 @@
           <state_interface name="position"/>
         </joint>
-        <joint name="${prefix}_front_right_mecanum_left_wheel_joint">
+        <joint name="${prefix}_wheel_RL_joint">
           <command_interface name="velocity">
             <param name="min">-10</param>
@@ -33,5 +33,5 @@
           <state_interface name="position"/>
         </joint>
-        <joint name="${prefix}_rear_right_mecanum_right_wheel_joint">
+        <joint name="${prefix}_wheel_RR_joint">
           <command_interface name="velocity">
             <param name="min">-10</param>
@@ -45,5 +45,5 @@
   requires a custom friction model so the vehicle can strafe left to right -->
       <!-- Wheel friction properties -->
-      <gazebo reference="${prefix}_rear_left_mecanum_left_wheel_link">
+      <gazebo reference="${prefix}_wheel_RL">
         <collision>
           <surface>
@@ -58,5 +58,5 @@
         </collision>
       </gazebo>
-      <gazebo reference="${prefix}_rear_right_mecanum_right_wheel_link">
+      <gazebo reference="${prefix}_wheel_RR">
         <collision>
           <surface>
@@ -71,5 +71,5 @@
         </collision>
       </gazebo>
-      <gazebo reference="${prefix}_front_left_mecanum_left_wheel_link">
+      <gazebo reference="${prefix}_wheel_FL">
         <collision>
           <surface>
@@ -84,5 +84,5 @@
         </collision>
       </gazebo>
-      <gazebo reference="${prefix}_front_right_mecanum_right_wheel_link">
+      <gazebo reference="${prefix}_wheel_FR">
         <collision>
           <surface>

File: home_custom_base_description/urdf/robot.xacro (robot description, xacro)
@@ -1,43 +1,223 @@
 <?xml version="1.0"?>
-<robot name="home_base"
-    xmlns:xacro="http://ros.org/wiki/xacro">
-    <!-- Launch arguments -->
-    <xacro:arg name="use_sim_time" default="true"/>
-    <xacro:arg name="robot_type" default="real"/>
-    <xacro:arg name="prefix" default="home_base"/>
-    <!-- Properties and Macros -->
-    <xacro:property name="name" default="home_base"/>
-    <xacro:property name="prefix" value="$(arg prefix)"/>
-    <xacro:property name="use_sim_time" value="$(arg use_sim_time)"/>
-    <!-- Include base description -->
-    <xacro:include filename="$(find home_custom_base_description)/urdf/inc/base.xacro"/>
-    <xacro:include filename="$(find home_custom_base_description)/urdf/inc/wheel.xacro"/>
-    <!-- Conditionally include simulation files -->
-    <xacro:if value="${use_sim_time}">
-        <xacro:include filename="$(find home_custom_base_description)/urdf/home_base_ros2_control.xacro"/>
-        <xacro:include filename="$(find home_custom_base_description)/urdf/home_base_gazebo.xacro"/>
-    </xacro:if>
-    <!-- Define base-->
-    <xacro:home_base_description name="${name}" prefix="${prefix}" />
-    <!-- Define wheel parent links -->
-    <xacro:property name="left_rear_parent_link" value="${prefix}_rear_left_wheel_frame"/>
-    <xacro:property name="right_rear_parent_link" value="${prefix}_rear_right_wheel_frame"/>
-    <xacro:property name="left_front_parent_link" value="${prefix}_front_left_wheel_frame"/>
-    <xacro:property name="right_front_parent_link" value="${prefix}_front_right_wheel_frame"/>
-    <!-- Define wheel connectors -->
-    <xacro:property name="connector_x_offset" value="0.0"/>
-    <xacro:property name="connector_y_offset" value="0.0"/>
-    <xacro:property name="connector_z_offset" value="0.015"/>
-    <!-- Define wheels -->
-    <xacro:home_base_wheel wheel_orientation="left" wheel_type="mecanum" parent_link="${left_rear_parent_link}" prefix="home_base_rear_left" x_offset="${connector_x_offset}" y_offset="${connector_y_offset}" z_offset="${connector_z_offset}" roll_offset="0.0" pitch_offset="0.0" yaw_offset="0.0" scale="0.001" axis_x="0" axis_y="0" axis_z="1" />
-    <xacro:home_base_wheel wheel_orientation="right" wheel_type="mecanum" parent_link="${right_rear_parent_link}" prefix="home_base_rear_right" x_offset="${connector_x_offset}" y_offset="${connector_y_offset}" z_offset="${-connector_z_offset}" roll_offset="0.0" pitch_offset="0.0" yaw_offset="0.0" scale="0.001" axis_x="0" axis_y="0" axis_z="1" />
-    <xacro:home_base_wheel wheel_orientation="left" wheel_type="mecanum" parent_link="${right_front_parent_link}" prefix="home_base_front_right" x_offset="${connector_x_offset}" y_offset="${connector_y_offset}" z_offset="${-connector_z_offset}" roll_offset="0.0" pitch_offset="0.0" yaw_offset="0.0" scale="0.001" axis_x="0" axis_y="0" axis_z="1" />
-    <xacro:home_base_wheel wheel_orientation="right" wheel_type="mecanum" parent_link="${left_front_parent_link}" prefix="home_base_front_left" x_offset="${connector_x_offset}" y_offset="${connector_y_offset}" z_offset="${connector_z_offset}" roll_offset="0.0" pitch_offset="0.0" yaw_offset="0.0" scale="0.001" axis_x="0" axis_y="0" axis_z="1" />
-    <!-- Conditionally add simulation components -->
-    <xacro:if value="${use_sim_time}">
-        <!-- Add ROS2 Control -->
-        <xacro:home_base_ros2_control name="${name}" prefix="${prefix}" use_sim_time="${use_sim_time}"/>
-        <!-- Add Gazebo simulation properties -->
-        <!-- <xacro:home_base_gazebo_sensors prefix="${prefix}"/> -->
-    </xacro:if>
+<robot name="home_base" xmlns:xacro="http://ros.org/wiki/xacro">
+  <!-- Launch arguments -->
+  <xacro:arg name="use_sim_time" default="true"/>
+  <xacro:arg name="robot_type" default="real"/>
+  <xacro:arg name="prefix" default="home_base"/>
+  <xacro:property name="prefix" value="$(arg prefix)"/>
+  <xacro:property name="use_sim_time" value="$(arg use_sim_time)"/>
+  <xacro:property name="mesh_dir" value="package://home_custom_base_description/meshes/visual"/>
+  <!-- Conditionally include simulation files -->
+  <xacro:if value="${use_sim_time}">
+    <xacro:include filename="$(find home_custom_base_description)/urdf/home_base_ros2_control.xacro"/>
+  </xacro:if>
+  <material name="home_base_gray">
+    <color rgba="0.752941176470588 0.752941176470588 0.752941176470588 1"/>
+  </material>
+  <material name="home_base_lidar">
+    <color rgba="0.792156862745098 0.819607843137255 0.933333333333333 1"/>
+  </material>
+  <!-- =================== base_footprint (root) =================== -->
+  <link name="${prefix}_base_footprint"/>
+  <joint name="${prefix}_base_footprint_joint" type="fixed">
+    <origin xyz="0 0 0.0385" rpy="0 0 0"/>
+    <parent link="${prefix}_base_footprint"/>
+    <child link="${prefix}_base_link"/>
+  </joint>
+  <!-- =================== base_link =================== -->
+  <link name="${prefix}_base_link">
+    <inertial>
+      <origin xyz="0.0323013333262494 -9.67443475711848E-05 0.199188228878544" rpy="0 0 0"/>
+      <mass value="23.590093490853"/>
+      <inertia ixx="0.132378675420004" ixy="1.47493862587287E-05" ixz="0.000807393658628412"
+               iyy="0.106153556594811" iyz="-9.34021230034792E-05" izz="0.166366947714662"/>
+    </inertial>
+    <visual>
+      <origin xyz="0 0 0" rpy="0 0 0"/>
+      <geometry>
+        <mesh filename="${mesh_dir}/base_link.STL"/>
+      </geometry>
+      <material name="home_base_gray"/>
+    </visual>
+    <collision>
+      <origin xyz="0 0 0" rpy="0 0 0"/>
+      <geometry>
+        <mesh filename="${mesh_dir}/base_link.STL"/>
+      </geometry>
+    </collision>
+  </link>
+  <!-- =================== wheel_FL =================== -->
+  <link name="${prefix}_wheel_FL">
+    <inertial>
+      <origin xyz="-2.01760275153617E-11 -1.2648801422932E-08 -0.000225751978378957" rpy="0 0 0"/>
+      <mass value="0.316522165409144"/>
+      <inertia ixx="0.00018550184297716" ixy="1.47011741018487E-13" ixz="2.37351682170515E-11"
+               iyy="0.000185501841925862" iyz="3.06630872791257E-11" izz="0.000329540832812286"/>
+    </inertial>
+    <visual>
+      <origin xyz="0 0 0" rpy="0 0 0"/>
+      <geometry>
+        <mesh filename="${mesh_dir}/wheel_FL.STL"/>
+      </geometry>
+      <material name="home_base_gray"/>
+    </visual>
+    <collision>
+      <origin xyz="0 0 0" rpy="0 0 0"/>
+      <geometry>
+        <mesh filename="${mesh_dir}/wheel_FL.STL"/>
+      </geometry>
+    </collision>
+  </link>
+  <joint name="${prefix}_wheel_FL_joint" type="continuous">
+    <origin xyz="0.184790699909997 0.219394995052441 0.0376959841787657" rpy="-1.5707963267949 0 0"/>
+    <parent link="${prefix}_base_link"/>
+    <child link="${prefix}_wheel_FL"/>
+    <axis xyz="0 0 1"/>
+  </joint>
+  <!-- =================== wheel_FR =================== -->
+  <link name="${prefix}_wheel_FR">
+    <inertial>
+      <origin xyz="1.08346649985158E-08 2.62530414074647E-09 -0.000243946115891319" rpy="0 0 0"/>
+      <mass value="0.316802369656036"/>
+      <inertia ixx="0.000185524626213339" ixy="3.28960054383515E-11" ixz="-3.31069057136383E-11"
+               iyy="0.000185524577692034" iyz="1.46274884608806E-10" izz="0.000329541494389925"/>
+    </inertial>
+    <visual>
+      <origin xyz="0 0 0" rpy="0 0 0"/>
+      <geometry>
+        <mesh filename="${mesh_dir}/wheel_FR.STL"/>
+      </geometry>
+      <material name="home_base_gray"/>
+    </visual>
+    <collision>
+      <origin xyz="0 0 0" rpy="0 0 0"/>
+      <geometry>
+        <mesh filename="${mesh_dir}/wheel_FR.STL"/>
+      </geometry>
+    </collision>
+  </link>
+  <joint name="${prefix}_wheel_FR_joint" type="continuous">
+    <origin xyz="0.184790699909996 -0.219395004947559 0.0376959841787653" rpy="-1.5707963267949 0 0"/>
+    <parent link="${prefix}_base_link"/>
+    <child link="${prefix}_wheel_FR"/>
+    <axis xyz="0 0 1"/>
+  </joint>
+  <!-- =================== wheel_RL =================== -->
+  <link name="${prefix}_wheel_RL">
+    <inertial>
+      <origin xyz="6.27955468179842E-09 -8.84368271322766E-09 -0.000243945799877326" rpy="0 0 0"/>
+      <mass value="0.316802379932942"/>
+      <inertia ixx="0.000185524613388858" ixy="-3.95566165674954E-11" ixz="1.17507787929333E-10"
+               iyy="0.000185524592122908" iyz="9.32696147810741E-11" izz="0.000329541494439521"/>
+    </inertial>
+    <visual>
+      <origin xyz="0 0 0" rpy="0 0 0"/>
+      <geometry>
+        <mesh filename="${mesh_dir}/wheel_RL.STL"/>
+      </geometry>
+      <material name="home_base_gray"/>
+    </visual>
+    <collision>
+      <origin xyz="0 0 0" rpy="0 0 0"/>
+      <geometry>
+        <mesh filename="${mesh_dir}/wheel_RL.STL"/>
+      </geometry>
+    </collision>
+  </link>
+  <joint name="${prefix}_wheel_RL_joint" type="continuous">
+    <origin xyz="-0.184790699909991 0.219394995052441 0.0376959841787652" rpy="-1.5707963267949 0 0"/>
+    <parent link="${prefix}_base_link"/>
+    <child link="${prefix}_wheel_RL"/>
+    <axis xyz="0 0 1"/>
+  </joint>
+  <!-- =================== wheel_RR =================== -->
+  <link name="${prefix}_wheel_RR">
+    <inertial>
+      <origin xyz="1.54742141322828E-09 1.26432938458987E-08 -0.000225751989580358" rpy="0 0 0"/>
+      <mass value="0.316522156157189"/>
+      <inertia ixx="0.000185501841998064" ixy="-9.89385955526853E-15" ixz="-2.625503122693E-11"
+               iyy="0.00018550184097349" iyz="-2.87014788963402E-11" izz="0.000329540832766985"/>
+    </inertial>
+    <visual>
+      <origin xyz="0 0 0" rpy="0 0 0"/>
+      <geometry>
+        <mesh filename="${mesh_dir}/wheel_RR.STL"/>
+      </geometry>
+      <material name="home_base_gray"/>
+    </visual>
+    <collision>
+      <origin xyz="0 0 0" rpy="0 0 0"/>
+      <geometry>
+        <mesh filename="${mesh_dir}/wheel_RR.STL"/>
+      </geometry>
+    </collision>
+  </link>
+  <joint name="${prefix}_wheel_RR_joint" type="continuous">
+    <origin xyz="-0.184790699909991 -0.219395004947559 0.0376959841787661" rpy="-1.5707963267949 0 0"/>
+    <parent link="${prefix}_base_link"/>
+    <child link="${prefix}_wheel_RR"/>
+    <axis xyz="0 0 1"/>
+  </joint>
+  <!-- =================== lidar_front =================== -->
+  <link name="${prefix}_lidar_front">
+    <inertial>
+      <origin xyz="-0.000159118177998852 3.36756577745678E-06 -0.00515345431268351" rpy="0 0 0"/>
+      <mass value="0.100467493631956"/>
+      <inertia ixx="3.42207960441524E-05" ixy="9.82554883966053E-09" ixz="-2.35749897825955E-07"
+               iyy="3.47512781108353E-05" iyz="4.57302960893946E-09" izz="4.25510359877868E-05"/>
+    </inertial>
+    <visual>
+      <origin xyz="0 0 0" rpy="0 0 0"/>
+      <geometry>
+        <mesh filename="${mesh_dir}/lidar_front.STL"/>
+      </geometry>
+      <material name="home_base_lidar"/>
+    </visual>
+    <collision>
+      <origin xyz="0 0 0" rpy="0 0 0"/>
+      <geometry>
+        <mesh filename="${mesh_dir}/lidar_front.STL"/>
+      </geometry>
+    </collision>
+  </link>
+  <joint name="${prefix}_lidar_front_joint" type="fixed">
+    <origin xyz="0.287749512711774 -0.207249957761446 0.135795984178765" rpy="0 0 -1.5707963267949"/>
+    <parent link="${prefix}_base_link"/>
+    <child link="${prefix}_lidar_front"/>
+  </joint>
+  <!-- =================== lidar_rear =================== -->
+  <link name="${prefix}_lidar_rear">
+    <inertial>
+      <origin xyz="-0.000159118177998907 3.36756577740127E-06 -0.00515345431268352" rpy="0 0 0"/>
+      <mass value="0.100467493631956"/>
+      <inertia ixx="3.42207960441524E-05" ixy="9.8255488396398E-09" ixz="-2.35749897825974E-07"
+               iyy="3.47512781108353E-05" iyz="4.57302960896798E-09" izz="4.25510359877867E-05"/>
+    </inertial>
+    <visual>
+      <origin xyz="0 0 0" rpy="0 0 0"/>
+      <geometry>
+        <mesh filename="${mesh_dir}/lidar_rear.STL"/>
+      </geometry>
+      <material name="home_base_lidar"/>
+    </visual>
+    <collision>
+      <origin xyz="0 0 0" rpy="0 0 0"/>
+      <geometry>
+        <mesh filename="${mesh_dir}/lidar_rear.STL"/>
+      </geometry>
+    </collision>
+  </link>
+  <joint name="${prefix}_lidar_rear_joint" type="fixed">
+    <origin xyz="-0.287749512711767 0.207249947866326 0.135795984178765" rpy="0 0 1.5707963267949"/>
+    <parent link="${prefix}_base_link"/>
+    <child link="${prefix}_lidar_rear"/>
+  </joint>
+  <!-- =================== Conditionally add simulation components =================== -->
+  <xacro:if value="${use_sim_time}">
+    <xacro:home_base_ros2_control name="home_base" prefix="${prefix}" use_sim_time="${use_sim_time}"/>
+    <!-- Webots driver plugin configuration -->
+    <webots>
+      <plugin type="webots_ros2_control::Ros2Control"/>
+    </webots>
+  </xacro:if>
 </robot>
