Commit message: delete unnecesary stls

File: home_custom_base_description/urdf/robot.xacro (robot description, xacro)
@@ -58,12 +58,12 @@
       <origin xyz="0 0 0" rpy="0 0 0"/>
       <geometry>
-        <mesh filename="${mesh_dir}/wheel_FL.STL"/>
-      </geometry>
-      <material name="home_base_gray"/>
-    </visual>
-    <collision>
-      <origin xyz="0 0 0" rpy="0 0 0"/>
-      <geometry>
-        <mesh filename="${mesh_dir}/wheel_FL.STL"/>
+        <mesh filename="${mesh_dir}/wheel.STL"/>
+      </geometry>
+      <material name="home_base_gray"/>
+    </visual>
+    <collision>
+      <origin xyz="0 0 0" rpy="0 0 0"/>
+      <geometry>
+        <mesh filename="${mesh_dir}/wheel.STL"/>
       </geometry>
     </collision>
@@ -86,12 +86,12 @@
       <origin xyz="0 0 0" rpy="0 0 0"/>
       <geometry>
-        <mesh filename="${mesh_dir}/wheel_FR.STL"/>
-      </geometry>
-      <material name="home_base_gray"/>
-    </visual>
-    <collision>
-      <origin xyz="0 0 0" rpy="0 0 0"/>
-      <geometry>
-        <mesh filename="${mesh_dir}/wheel_FR.STL"/>
+        <mesh filename="${mesh_dir}/wheel.STL"/>
+      </geometry>
+      <material name="home_base_gray"/>
+    </visual>
+    <collision>
+      <origin xyz="0 0 0" rpy="0 0 0"/>
+      <geometry>
+        <mesh filename="${mesh_dir}/wheel.STL"/>
       </geometry>
     </collision>
@@ -114,12 +114,12 @@
       <origin xyz="0 0 0" rpy="0 0 0"/>
       <geometry>
-        <mesh filename="${mesh_dir}/wheel_RL.STL"/>
-      </geometry>
-      <material name="home_base_gray"/>
-    </visual>
-    <collision>
-      <origin xyz="0 0 0" rpy="0 0 0"/>
-      <geometry>
-        <mesh filename="${mesh_dir}/wheel_RL.STL"/>
+        <mesh filename="${mesh_dir}/wheel.STL"/>
+      </geometry>
+      <material name="home_base_gray"/>
+    </visual>
+    <collision>
+      <origin xyz="0 0 0" rpy="0 0 0"/>
+      <geometry>
+        <mesh filename="${mesh_dir}/wheel.STL"/>
       </geometry>
     </collision>
@@ -142,12 +142,12 @@
       <origin xyz="0 0 0" rpy="0 0 0"/>
       <geometry>
-        <mesh filename="${mesh_dir}/wheel_RR.STL"/>
-      </geometry>
-      <material name="home_base_gray"/>
-    </visual>
-    <collision>
-      <origin xyz="0 0 0" rpy="0 0 0"/>
-      <geometry>
-        <mesh filename="${mesh_dir}/wheel_RR.STL"/>
+        <mesh filename="${mesh_dir}/wheel.STL"/>
+      </geometry>
+      <material name="home_base_gray"/>
+    </visual>
+    <collision>
+      <origin xyz="0 0 0" rpy="0 0 0"/>
+      <geometry>
+        <mesh filename="${mesh_dir}/wheel.STL"/>
       </geometry>
     </collision>

Commit message: update URDF with more detailed stl and turned xarm base

File: home_custom_base_description/urdf/robot.xacro (robot description, xacro)
@@ -28,8 +28,8 @@
   <link name="${prefix}_base_link">
     <inertial>
-      <origin xyz="0.0323013333262494 -9.67443475711848E-05 0.199188228878544" rpy="0 0 0"/>
-      <mass value="23.590093490853"/>
-      <inertia ixx="0.132378675420004" ixy="1.47493862587287E-05" ixz="0.000807393658628412"
-               iyy="0.106153556594811" iyz="-9.34021230034792E-05" izz="0.166366947714662"/>
+      <origin xyz="0.0035289 4.9532E-05 0.18881" rpy="0 0 0"/>
+      <mass value="31.284"/>
+      <inertia ixx="0.16472" ixy="6.3557E-05" ixz="0.00075615"
+               iyy="0.12042" iyz="-0.0002185" izz="0.20341"/>
     </inertial>
     <visual>
@@ -212,4 +212,11 @@
     <parent link="${prefix}_base_link"/>
     <child link="${prefix}_lidar_rear"/>
+  </joint>
+  <link name="xarm_base" />
+  <joint name="xarm_joint" type="fixed">
+    <origin xyz="0.0410000000000036 -0.00367166302995694 0.520695984178765" rpy="0 0 0" />
+    <parent link="${prefix}_base_link" />
+    <child link="xarm_base" />
+    <axis xyz="0 0 0" />
   </joint>
   <!-- =================== Conditionally add simulation components =================== -->

Commit message: refactor: standardize URDF link naming, update lidar orientations, add IMU frame, and introduce navigation basics launch file

File: home_custom_base_description/urdf/robot.xacro (robot description, xacro)
@@ -2,9 +2,11 @@
 <robot name="home_base" xmlns:xacro="http://ros.org/wiki/xacro">
   <!-- Launch arguments -->
-  <xacro:arg name="use_sim_time" default="true"/>
+  <xacro:arg name="use_sim_time" default="false"/>
   <xacro:arg name="robot_type" default="real"/>
-  <xacro:arg name="prefix" default="home_base"/>
+  <xacro:arg name="prefix" default=""/>
+  <xacro:arg name="imu_frame" default="imu_link"/>
   <xacro:property name="prefix" value="$(arg prefix)"/>
   <xacro:property name="use_sim_time" value="$(arg use_sim_time)"/>
+  <xacro:property name="imu_frame" value="$(arg imu_frame)"/>
   <xacro:property name="mesh_dir" value="package://home_custom_base_description/meshes/visual"/>
   <!-- Conditionally include simulation files -->
@@ -19,12 +21,12 @@
   </material>
   <!-- =================== base_footprint (root) =================== -->
-  <link name="${prefix}_base_footprint"/>
-  <joint name="${prefix}_base_footprint_joint" type="fixed">
+  <link name="${prefix}base_footprint"/>
+  <joint name="${prefix}base_footprint_joint" type="fixed">
     <origin xyz="0 0 0.0385" rpy="0 0 0"/>
-    <parent link="${prefix}_base_footprint"/>
-    <child link="${prefix}_base_link"/>
+    <parent link="${prefix}base_footprint"/>
+    <child link="${prefix}base_link"/>
   </joint>
   <!-- =================== base_link =================== -->
-  <link name="${prefix}_base_link">
+  <link name="${prefix}base_link">
     <inertial>
       <origin xyz="0.0323013333262494 -9.67443475711848E-05 0.199188228878544" rpy="0 0 0"/>
@@ -48,5 +50,5 @@
   </link>
   <!-- =================== wheel_FL =================== -->
-  <link name="${prefix}_wheel_FL">
+  <link name="${prefix}wheel_FL">
     <inertial>
       <origin xyz="-2.01760275153617E-11 -1.2648801422932E-08 -0.000225751978378957" rpy="0 0 0"/>
@@ -71,10 +73,10 @@
   <joint name="${prefix}_wheel_FL_joint" type="continuous">
     <origin xyz="0.184790699909997 0.219394995052441 0.0376959841787657" rpy="-1.5707963267949 0 0"/>
-    <parent link="${prefix}_base_link"/>
-    <child link="${prefix}_wheel_FL"/>
+    <parent link="${prefix}base_link"/>
+    <child link="${prefix}wheel_FL"/>
     <axis xyz="0 0 1"/>
   </joint>
   <!-- =================== wheel_FR =================== -->
-  <link name="${prefix}_wheel_FR">
+  <link name="${prefix}wheel_FR">
     <inertial>
       <origin xyz="1.08346649985158E-08 2.62530414074647E-09 -0.000243946115891319" rpy="0 0 0"/>
@@ -97,12 +99,12 @@
     </collision>
   </link>
-  <joint name="${prefix}_wheel_FR_joint" type="continuous">
+  <joint name="${prefix}wheel_FR_joint" type="continuous">
     <origin xyz="0.184790699909996 -0.219395004947559 0.0376959841787653" rpy="-1.5707963267949 0 0"/>
-    <parent link="${prefix}_base_link"/>
-    <child link="${prefix}_wheel_FR"/>
+    <parent link="${prefix}base_link"/>
+    <child link="${prefix}wheel_FR"/>
     <axis xyz="0 0 1"/>
   </joint>
   <!-- =================== wheel_RL =================== -->
-  <link name="${prefix}_wheel_RL">
+  <link name="${prefix}wheel_RL">
     <inertial>
       <origin xyz="6.27955468179842E-09 -8.84368271322766E-09 -0.000243945799877326" rpy="0 0 0"/>
@@ -125,12 +127,12 @@
     </collision>
   </link>
-  <joint name="${prefix}_wheel_RL_joint" type="continuous">
+  <joint name="${prefix}wheel_RL_joint" type="continuous">
     <origin xyz="-0.184790699909991 0.219394995052441 0.0376959841787652" rpy="-1.5707963267949 0 0"/>
-    <parent link="${prefix}_base_link"/>
-    <child link="${prefix}_wheel_RL"/>
+    <parent link="${prefix}base_link"/>
+    <child link="${prefix}wheel_RL"/>
     <axis xyz="0 0 1"/>
   </joint>
   <!-- =================== wheel_RR =================== -->
-  <link name="${prefix}_wheel_RR">
+  <link name="${prefix}wheel_RR">
     <inertial>
       <origin xyz="1.54742141322828E-09 1.26432938458987E-08 -0.000225751989580358" rpy="0 0 0"/>
@@ -153,12 +155,12 @@
     </collision>
   </link>
-  <joint name="${prefix}_wheel_RR_joint" type="continuous">
+  <joint name="${prefix}wheel_RR_joint" type="continuous">
     <origin xyz="-0.184790699909991 -0.219395004947559 0.0376959841787661" rpy="-1.5707963267949 0 0"/>
-    <parent link="${prefix}_base_link"/>
-    <child link="${prefix}_wheel_RR"/>
+    <parent link="${prefix}base_link"/>
+    <child link="${prefix}wheel_RR"/>
     <axis xyz="0 0 1"/>
   </joint>
   <!-- =================== lidar_front =================== -->
-  <link name="${prefix}_lidar_front">
+  <link name="${prefix}lidar_front">
     <inertial>
       <origin xyz="-0.000159118177998852 3.36756577745678E-06 -0.00515345431268351" rpy="0 0 0"/>
@@ -181,11 +183,11 @@
     </collision>
   </link>
-  <joint name="${prefix}_lidar_front_joint" type="fixed">
-    <origin xyz="0.287749512711774 -0.207249957761446 0.135795984178765" rpy="0 0 -1.5707963267949"/>
-    <parent link="${prefix}_base_link"/>
-    <child link="${prefix}_lidar_front"/>
+  <joint name="${prefix}lidar_front_joint" type="fixed">
+    <origin xyz="0.287749512711774 -0.207249957761446 0.135795984178765" rpy="0 0 1.57"/>
+    <parent link="${prefix}base_link"/>
+    <child link="${prefix}lidar_front"/>
   </joint>
   <!-- =================== lidar_rear =================== -->
-  <link name="${prefix}_lidar_rear">
+  <link name="${prefix}lidar_rear">
     <inertial>
       <origin xyz="-0.000159118177998907 3.36756577740127E-06 -0.00515345431268352" rpy="0 0 0"/>
@@ -208,8 +210,16 @@
     </collision>
   </link>
-  <joint name="${prefix}_lidar_rear_joint" type="fixed">
-    <origin xyz="-0.287749512711767 0.207249947866326 0.135795984178765" rpy="0 0 1.5707963267949"/>
-    <parent link="${prefix}_base_link"/>
-    <child link="${prefix}_lidar_rear"/>
+  <joint name="${prefix}lidar_rear_joint" type="fixed">
+    <origin xyz="-0.287749512711767 0.207249947866326 0.135795984178765" rpy="0 0 -1.57"/>
+    <parent link="${prefix}base_link"/>
+    <child link="${prefix}lidar_rear"/>
+  </joint>
+  <!-- =================== imu (base_link -> imu_frame) =================== -->
+  <!-- Replaces the base_to_imu static_transform_publisher node -->
+  <link name="${prefix}${imu_frame}"/>
+  <joint name="${prefix}base_to_imu" type="fixed">
+    <origin xyz="0 0 0" rpy="0 0 0"/>
+    <parent link="${prefix}base_link"/>
+    <child link="${prefix}${imu_frame}"/>
   </joint>
   <!-- =================== Conditionally add simulation components =================== -->
